Commit message: Fix OmniHand visual asset loading

File: source/atec_rl_lab/atec_rl_lab/assets/robots/o12_hand_description-o12_t3/assets/urdf/omnihand_pro_left.urdf (robot description, URDF)
Before this commit: robot omnihand_pro_left, 26 links, 25 joints
Links:
- link L_index_abad_link: geometry visual mesh filename=../meshes/index_abad.STL
- link L_index_dip_link: geometry collision cylinder length=0.02 radius=0.01; visual mesh filename=../meshes/finger_dip.STL
- link L_index_mcp_link: geometry collision cylinder length=0.038 radius=0.01; visual mesh filename=../meshes/index_mcp.STL
- link L_index_pip_link: geometry collision cylinder length=0.022 radius=0.01; visual mesh filename=../meshes/index_pip.STL
- link L_middle_abad_link: geometry visual mesh filename=../meshes/middle_abad.STL
- link L_middle_dip_link: geometry collision cylinder length=0.018 radius=0.01; visual mesh filename=../meshes/finger_dip.STL
- link L_middle_mcp_link: geometry collision cylinder length=0.04 radius=0.01; visual mesh filename=../meshes/middle_mcp.STL
- link L_middle_pip_link: geometry collision cylinder length=0.028 radius=0.01; visual mesh filename=../meshes/middle_pip.STL
- link L_palm: geometry collision box size=0.05 0.09 0.09; collision cylinder length=0.01 radius=0.032
- link L_pinky_dip_link: geometry collision cylinder length=0.018 radius=0.01; visual mesh filename=../meshes/finger_dip.STL
- link L_pinky_mcp_link: geometry collision cylinder length=0.035 radius=0.01; visual mesh filename=../meshes/ring_mcp.STL
- link L_pinky_pip_link: geometry collision cylinder length=0.028 radius=0.01; visual mesh filename=../meshes/ring_pip.STL
- link L_ring_dip_link: geometry collision cylinder length=0.018 radius=0.01; visual mesh filename=../meshes/finger_dip.STL
- link L_ring_mcp_link: geometry collision cylinder length=0.035 radius=0.01; visual mesh filename=../meshes/ring_mcp.STL
- link L_ring_pip_link: geometry collision cylinder length=0.028 radius=0.01; visual mesh filename=../meshes/ring_pip.STL
- link L_thumb_abad_link: geometry collision box size=0.035 0.006 0.02; visual mesh filename=../meshes/l_thumb_abad.STL
- link L_thumb_dip_link: geometry collision cylinder length=0.03 radius=0.01; visual mesh filename=../meshes/thumb_dip.STL
- link L_thumb_mcp_link: geometry collision box size=0.064 0.023 0.03; visual mesh filename=../meshes/thumb_mcp.STL
- link L_thumb_pip_link: geometry collision cylinder length=0.02 radius=0.01; visual mesh filename=../meshes/thumb_pip.STL
- link L_thumb_roll_link: geometry visual mesh filename=../meshes/l_thumb_roll.STL

File: source/atec_rl_lab/atec_rl_lab/assets/robots/o12_hand_description-o12_t3/assets/urdf/omnihand_pro_right.urdf (robot description, URDF)
Before this commit: robot omnihand_pro_right, 26 links, 25 joints
Links:
- link R_index_abad_link: geometry visual mesh filename=../meshes/index_abad.STL
- link R_index_dip_link: geometry collision cylinder length=0.02 radius=0.01; visual mesh filename=../meshes/finger_dip.STL
- link R_index_mcp_link: geometry collision cylinder length=0.038 radius=0.01; visual mesh filename=../meshes/index_mcp.STL
- link R_index_pip_link: geometry collision cylinder length=0.022 radius=0.01; visual mesh filename=../meshes/index_pip.STL
- link R_middle_abad_link: geometry visual mesh filename=../meshes/middle_abad.STL
- link R_middle_dip_link: geometry collision cylinder length=0.018 radius=0.01; visual mesh filename=../meshes/finger_dip.STL
- link R_middle_mcp_link: geometry collision cylinder length=0.04 radius=0.01; visual mesh filename=../meshes/middle_mcp.STL
- link R_middle_pip_link: geometry collision cylinder length=0.028 radius=0.01; visual mesh filename=../meshes/middle_pip.STL
- link R_palm: geometry collision box size=0.05 0.09 0.09; collision cylinder length=0.01 radius=0.032
- link R_pinky_dip_link: geometry collision cylinder length=0.018 radius=0.01; visual mesh filename=../meshes/finger_dip.STL
- link R_pinky_mcp_link: geometry collision cylinder length=0.035 radius=0.01; visual mesh filename=../meshes/ring_mcp.STL
- link R_pinky_pip_link: geometry collision cylinder length=0.028 radius=0.01; visual mesh filename=../meshes/ring_pip.STL
- link R_ring_dip_link: geometry collision cylinder length=0.018 radius=0.01; visual mesh filename=../meshes/finger_dip.STL
- link R_ring_mcp_link: geometry collision cylinder length=0.035 radius=0.01; visual mesh filename=../meshes/ring_mcp.STL
- link R_ring_pip_link: geometry collision cylinder length=0.028 radius=0.01; visual mesh filename=../meshes/ring_pip.STL
- link R_thumb_abad_link: geometry collision box size=0.035 0.006 0.02; visual mesh filename=../meshes/r_thumb_abad.STL
- link R_thumb_dip_link: geometry collision cylinder length=0.03 radius=0.01; visual mesh filename=../meshes/thumb_dip.STL
- link R_thumb_mcp_link: geometry collision box size=0.064 0.023 0.03; visual mesh filename=../meshes/thumb_mcp.STL
- link R_thumb_pip_link: geometry collision cylinder length=0.02 radius=0.01; visual mesh filename=../meshes/thumb_pip.STL
- link R_thumb_roll_link: geometry visual mesh filename=../meshes/r_thumb_roll.STL

File: source/atec_rl_lab/atec_rl_lab/assets/robots/o12_hand_description-o12_t3/assets/urdf_mesh_col/omnihand_pro_left.urdf (robot description, URDF)
Before this commit: robot omnihand_pro_left, 26 links, 25 joints
Links:
- link L_index_abad_link: geometry visual mesh filename=../meshes/index_abad.STL
- link L_index_dip_link: geometry collision mesh filename=../meshes/collision/finger_dip_col.STL; visual mesh filename=../meshes/finger_dip.STL
- link L_index_mcp_link: geometry collision mesh filename=../meshes/collision/index_mcp_col.STL; visual mesh filename=../meshes/index_mcp.STL
- link L_index_pip_link: geometry collision mesh filename=../meshes/collision/index_pip_col.STL; visual mesh filename=../meshes/index_pip.STL
- link L_middle_abad_link: geometry visual mesh filename=../meshes/middle_abad.STL
- link L_middle_dip_link: geometry collision mesh filename=../meshes/collision/finger_dip_col.STL; visual mesh filename=../meshes/finger_dip.STL
- link L_middle_mcp_link: geometry collision mesh filename=../meshes/collision/middle_mcp_col.STL; visual mesh filename=../meshes/middle_mcp.STL
- link L_middle_pip_link: geometry collision mesh filename=../meshes/collision/middle_pip_col.STL; visual mesh filename=../meshes/middle_pip.STL
- link L_palm: geometry collision mesh filename=../meshes/collision/l_palm_col.STL; visual mesh filename=../meshes/l_palm.STL
- link L_pinky_dip_link: geometry collision mesh filename=../meshes/collision/finger_dip_col.STL; visual mesh filename=../meshes/finger_dip.STL
- link L_pinky_mcp_link: geometry collision mesh filename=../meshes/collision/ring_mcp_col.STL; visual mesh filename=../meshes/ring_mcp.STL
- link L_pinky_pip_link: geometry collision mesh filename=../meshes/collision/ring_pip_col.STL; visual mesh filename=../meshes/ring_pip.STL
- link L_ring_dip_link: geometry collision mesh filename=../meshes/collision/finger_dip_col.STL; visual mesh filename=../meshes/finger_dip.STL
- link L_ring_mcp_link: geometry collision mesh filename=../meshes/collision/ring_mcp_col.STL; visual mesh filename=../meshes/ring_mcp.STL
- link L_ring_pip_link: geometry collision mesh filename=../meshes/collision/ring_pip_col.STL; visual mesh filename=../meshes/ring_pip.STL
- link L_thumb_abad_link: geometry collision mesh filename=../meshes/collision/l_thumb_abad_col.STL; visual mesh filename=../meshes/l_thumb_abad.STL
- link L_thumb_dip_link: geometry collision mesh filename=../meshes/collision/thumb_dip_col.STL; visual mesh filename=../meshes/thumb_dip.STL
- link L_thumb_mcp_link: geometry collision mesh filename=../meshes/collision/thumb_mcp_col.STL; visual mesh filename=../meshes/thumb_mcp.STL
- link L_thumb_pip_link: geometry collision mesh filename=../meshes/collision/thumb_pip_col.STL; visual mesh filename=../meshes/thumb_pip.STL
- link L_thumb_roll_link: geometry collision mesh filename=../meshes/collision/l_thumb_roll_col.STL; visual mesh filename=../meshes/l_thumb_roll.STL

File: source/atec_rl_lab/atec_rl_lab/assets/robots/o12_hand_description-o12_t3/assets/urdf_mesh_col/omnihand_pro_right.urdf (robot description, URDF)
Before this commit: robot omnihand_pro_right, 26 links, 25 joints
Links:
- link R_index_abad_link: geometry visual mesh filename=../meshes/index_abad.STL
- link R_index_dip_link: geometry collision mesh filename=../meshes/collision/finger_dip_col.STL; visual mesh filename=../meshes/finger_dip.STL
- link R_index_mcp_link: geometry collision mesh filename=../meshes/collision/index_mcp_col.STL; visual mesh filename=../meshes/index_mcp.STL
- link R_index_pip_link: geometry collision mesh filename=../meshes/collision/index_pip_col.STL; visual mesh filename=../meshes/index_pip.STL
- link R_middle_abad_link: geometry visual mesh filename=../meshes/middle_abad.STL
- link R_middle_dip_link: geometry collision mesh filename=../meshes/collision/finger_dip_col.STL; visual mesh filename=../meshes/finger_dip.STL
- link R_middle_mcp_link: geometry collision mesh filename=../meshes/collision/middle_mcp_col.STL; visual mesh filename=../meshes/middle_mcp.STL
- link R_middle_pip_link: geometry collision mesh filename=../meshes/collision/middle_pip_col.STL; visual mesh filename=../meshes/middle_pip.STL
- link R_palm: geometry collision mesh filename=../meshes/collision/r_palm_col.STL; visual mesh filename=../meshes/r_palm.STL
- link R_pinky_dip_link: geometry collision mesh filename=../meshes/collision/finger_dip_col.STL; visual mesh filename=../meshes/finger_dip.STL
- link R_pinky_mcp_link: geometry collision mesh filename=../meshes/collision/ring_mcp_col.STL; visual mesh filename=../meshes/ring_mcp.STL
- link R_pinky_pip_link: geometry collision mesh filename=../meshes/collision/ring_pip_col.STL; visual mesh filename=../meshes/ring_pip.STL
- link R_ring_dip_link: geometry collision mesh filename=../meshes/collision/finger_dip_col.STL; visual mesh filename=../meshes/finger_dip.STL
- link R_ring_mcp_link: geometry collision mesh filename=../meshes/collision/ring_mcp_col.STL; visual mesh filename=../meshes/ring_mcp.STL
- link R_ring_pip_link: geometry collision mesh filename=../meshes/collision/ring_pip_col.STL; visual mesh filename=../meshes/ring_pip.STL
- link R_thumb_abad_link: geometry collision mesh filename=../meshes/collision/r_thumb_abad_col.STL; visual mesh filename=../meshes/r_thumb_abad.STL
- link R_thumb_dip_link: geometry collision mesh filename=../meshes/collision/thumb_dip_col.STL; visual mesh filename=../meshes/thumb_dip.STL
- link R_thumb_mcp_link: geometry collision mesh filename=../meshes/collision/thumb_mcp_col.STL; visual mesh filename=../meshes/thumb_mcp.STL
- link R_thumb_pip_link: geometry collision mesh filename=../meshes/collision/thumb_pip_col.STL; visual mesh filename=../meshes/thumb_pip.STL
- link R_thumb_roll_link: geometry collision mesh filename=../meshes/collision/r_thumb_roll_col.STL; visual mesh filename=../meshes/r_thumb_roll.STL

Commit message: collision

File: source/atec_rl_lab/atec_rl_lab/assets/robots/o12_hand_description-o12_t3/assets/urdf/omnihand_pro_left.urdf (robot description, URDF)
Before this commit: robot omnihand_pro_left, 26 links, 25 joints
Links:
- link L_thumb_abad_link: geometry visual mesh filename=../meshes/l_thumb_abad.STL
